Commit message: update new base model

File: workspace/src/hsa_bot/urdf/hsa_bot.xacro (robot description, xacro)
@@ -2,195 +2,356 @@
 <robot name="hsa_bot" xmlns:xacro="http://www.ros.org/wiki/xacro">
   <xacro:include filename="$(find hsa_bot)/urdf/hsa_bot.gazebo" />
-  <link name="robot_footprint"></link>
-  <joint name="robot_footprint_joint" type="fixed">
+<link name="robot_footprint">
+   <visual>
+      <origin xyz="0 0 0" rpy="0 0 0" />
+      <geometry>
+        <box size="0.001 0.001 0.001" />
+      </geometry>
+    </visual>
+  </link>
+  <joint name="base_link_joint" type="fixed">
     <origin xyz="0 0 0" rpy="0 0 0" />
     <parent link="robot_footprint"/>
     <child link="base_link" />
   </joint>
-  <link name='base_link'>
-    <pose>0 0 0.1 0 0 0</pose>
-    <inertial>
-      <mass value="15.0"/>
-      <origin xyz="0.0 0 0" rpy=" 0 0 0"/>
-      <inertia
-          ixx="0.1" ixy="0" ixz="0"
-          iyy="0.1" iyz="0"
-          izz="0.1"
-      />
-    </inertial>
-    <collision name='collision'>
-      <origin xyz="0 0 0" rpy=" 0 0 0"/>
-      <geometry>
-        <box size=".4 .2 .1"/>
-      </geometry>
-    </collision>
-    <visual name='base_link_visual'>
-      <origin xyz="0 0 0" rpy=" 0 0 0"/>
-      <geometry>
-        <box size=".4 .2 .1"/>
-      </geometry>
-    </visual>
-    <collision name='back_caster_collision'>
-      <origin xyz="-0.15 0 -0.05" rpy=" 0 0 0"/>
-      <geometry>
-        <sphere radius="0.0499"/>
-      </geometry>
-      <surface>
-        <friction>
-          <ode>
-            <mu>0</mu>
-            <mu2>0</mu2>
-            <slip1>1.0</slip1>
-            <slip2>1.0</slip2>
-          </ode>
-        </friction>
-      </surface>
-    </collision>
-    <visual name='back_caster_visual'>
-      <origin xyz="-0.15 0 -0.05" rpy=" 0 0 0"/>
-      <geometry>
-        <sphere radius="0.05"/>
-      </geometry>
-    </visual>
-    <collision name='front_caster_collision'>
-      <origin xyz="0.15 0 -0.05" rpy=" 0 0 0"/>
-      <geometry>
-        <sphere radius="0.0499"/>
-      </geometry>
-      <surface>
-        <friction>
-          <ode>
-            <mu>0</mu>
-            <mu2>0</mu2>
-            <slip1>1.0</slip1>
-            <slip2>1.0</slip2>
-          </ode>
-        </friction>
-      </surface>
-    </collision>
-    <visual name='front_caster_visual'>
-      <origin xyz="0.15 0 -0.05" rpy=" 0 0 0"/>
-      <geometry>
-        <sphere radius="0.05"/>
-      </geometry>
-    </visual>
-  </link>
-  <link name="left_wheel">
-    <inertial>
-      <mass value="5.0"/>
-      <origin xyz="0 0 0" rpy=" 0 1.5707 1.5707"/>
-      <inertia
-          ixx="0.1" ixy="0" ixz="0"
-          iyy="0.1" iyz="0"
-          izz="0.1"
-      />
-    </inertial>
-    <collision name='left_wheel_collision'>
-      <origin xyz="0 0 0" rpy=" 0 1.5707 1.5707"/>
-      <geometry>
-        <cylinder radius="0.1" length="0.05" />
-      </geometry>
-    </collision>
-    <visual name='left_wheel_visual'>
-      <origin xyz="0 0 0" rpy=" 0 1.5707 1.5707"/>
-      <geometry>
-        <cylinder radius="0.1" length="0.05" />
-      </geometry>
-    </visual>
-  </link>
-  <link name="right_wheel">
-    <inertial>
-      <mass value="5.0"/>
-      <origin xyz="0 0 0" rpy=" 0 1.5707 1.5707"/>
-      <inertia
-          ixx="0.1" ixy="0" ixz="0"
-          iyy="0.1" iyz="0"
-          izz="0.1"
-      />
-    </inertial>
-    <collision name='right_wheel_collision'>
-      <origin xyz="0 0 0" rpy=" 0 1.5707 1.5707"/>
-      <geometry>
-        <cylinder radius="0.1" length="0.05" />
-      </geometry>
-    </collision>
-    <visual name='right_wheel_visual'>
-      <origin xyz="0 0 0" rpy=" 0 1.5707 1.5707"/>
-      <geometry>
-        <cylinder radius="0.1" length="0.05" />
-      </geometry>
-    </visual>
-  </link>
-  <joint type="continuous" name="left_wheel_hinge">
-    <origin xyz="0 0.15 0" rpy="0 0 0"/>
-    <child link="left_wheel"/>
+  <link
+    name="base_link">
+    <inertial>
+      <origin
+        xyz="0 0 0.04"
+        rpy="0 0 0" />
+      <mass
+        value="0.59313" />
+      <inertia
+        ixx="0.0013364"
+        ixy="4.824E-20"
+        ixz="1.7974E-21"
+        iyy="0.0038545"
+        iyz="3.8567E-21"
+        izz="0.0051839" />
+    </inertial>
+    <visual>
+      <origin
+        xyz="0 0 0"
+        rpy="0 0 0" />
+      <geometry>
+        <mesh
+          filename="package://hsa_bot/meshes/base_link.STL" />
+      </geometry>
+      <material
+        name="">
+        <color
+          rgba="1 1 1 1" />
+      </material>
+    </visual>
+    <collision>
+      <origin
+        xyz="0 0 0"
+        rpy="0 0 0" />
+      <geometry>
+        <mesh
+          filename="package://hsa_bot/meshes/base_link.STL" />
+      </geometry>
+    </collision>
+  </link>
+  <link
+    name="link_wheel_FL">
+    <inertial>
+      <origin
+        xyz="0 0.012 0"
+        rpy="0 0 0" />
+      <mass
+        value="0.10053" />
+      <inertia
+        ixx="4.3563E-05"
+        ixy="1.1294E-21"
+        ixz="-1.6941E-21"
+        iyy="8.0425E-05"
+        iyz="-7.0586E-23"
+        izz="4.3563E-05" />
+    </inertial>
+    <visual>
+      <origin
+        xyz="0 0 0"
+        rpy="0 0 0" />
+      <geometry>
+        <mesh
+          filename="package://hsa_bot/meshes/link_wheel_FL.STL" />
+      </geometry>
+      <material
+        name="">
+        <color
+          rgba="1 1 1 1" />
+      </material>
+    </visual>
+    <collision>
+      <origin
+        xyz="0 0 0"
+        rpy="0 0 0" />
+      <geometry>
+        <mesh
+          filename="package://hsa_bot/meshes/link_wheel_FL.STL" />
+      </geometry>
+    </collision>
+  </link>
+  <joint
+    name="joint_wheel_FL"
+    type="continuous">
+    <origin
+      xyz="0.08 0.08 0.04"
+      rpy="0 0 0" />
+    <parent
+      link="base_link" />
+    <child
+      link="link_wheel_FL" />
+    <axis
+      xyz="0 1 0" />
+  </joint>
+  <link
+    name="link_wheel_FR">
+    <inertial>
+      <origin
+        xyz="0 -0.012 0"
+        rpy="0 0 0" />
+      <mass
+        value="0.10053" />
+      <inertia
+        ixx="4.3563E-05"
+        ixy="-7.2158E-38"
+        ixz="-5.294E-23"
+        iyy="8.0425E-05"
+        iyz="7.9908E-38"
+        izz="4.3563E-05" />
+    </inertial>
+    <visual>
+      <origin
+        xyz="0 0 0"
+        rpy="0 0 0" />
+      <geometry>
+        <mesh
+          filename="package://hsa_bot/meshes/link_wheel_FR.STL" />
+      </geometry>
+      <material
+        name="">
+        <color
+          rgba="1 1 1 1" />
+      </material>
+    </visual>
+    <collision>
+      <origin
+        xyz="0 0 0"
+        rpy="0 0 0" />
+      <geometry>
+        <mesh
+          filename="package://hsa_bot/meshes/link_wheel_FR.STL" />
+      </geometry>
+    </collision>
+  </link>
+  <joint
+    name="joint_wheel_FR"
+    type="continuous">
+    <origin
+      xyz="0.0800000000000013 -0.0799999999999997 0.04"
+      rpy="0 0 0" />
+    <parent
+      link="base_link" />
+    <child
+      link="link_wheel_FR" />
+    <axis
+      xyz="0 1 0" />
+  </joint>
+  <link
+    name="link_wheel_BL">
+    <inertial>
+      <origin
+        xyz="0 0.012 0"
+        rpy="0 0 0" />
+      <mass
+        value="0.10053" />
+      <inertia
+        ixx="4.3563E-05"
+        ixy="5.6469E-22"
+        ixz="5.6469E-22"
+        iyy="8.0425E-05"
+        iyz="-4.2977E-37"
+        izz="4.3563E-05" />
+    </inertial>
+    <visual>
+      <origin
+        xyz="0 0 0"
+        rpy="0 0 0" />
+      <geometry>
+        <mesh
+          filename="package://hsa_bot/meshes/link_wheel_BL.STL" />
+      </geometry>
+      <material
+        name="">
+        <color
+          rgba="1 1 1 1" />
+      </material>
+    </visual>
+    <collision>
+      <origin
+        xyz="0 0 0"
+        rpy="0 0 0" />
+      <geometry>
+        <mesh
+          filename="package://hsa_bot/meshes/link_wheel_BL.STL" />
+      </geometry>
+    </collision>
+  </link>
+  <joint
+    name="joint_wheel_BL"
+    type="continuous">
+    <origin
+      xyz="-0.08 0.08 0.04"
+      rpy="0 0 0" />
+    <parent
+      link="base_link" />
+    <child
+      link="link_wheel_BL" />
+    <axis
+      xyz="0 1 0" />
+  </joint>
+  <link
+    name="link_wheel_BR">
+    <inertial>
+      <origin
+        xyz="0 -0.012 0"
+        rpy="0 0 0" />
+      <mass
+        value="0.10053" />
+      <inertia
+        ixx="4.3563E-05"
+        ixy="-7.3468E-38"
+        ixz="-6.1763E-23"
+        iyy="8.0425E-05"
+        iyz="-4.5918E-39"
+        izz="4.3563E-05" />
+    </inertial>
+    <visual>
+      <origin
+        xyz="0 0 0"
+        rpy="0 0 0" />
+      <geometry>
+        <mesh
+          filename="package://hsa_bot/meshes/link_wheel_BR.STL" />
+      </geometry>
+      <material
+        name="">
+        <color
+          rgba="1 1 1 1" />
+      </material>
+    </visual>
+    <collision>
+      <origin
+        xyz="0 0 0"
+        rpy="0 0 0" />
+      <geometry>
+        <mesh
+          filename="package://hsa_bot/meshes/link_wheel_BR.STL" />
+      </geometry>
+    </collision>
+  </link>
+  <joint
+    name="joint_wheel_BR"
+    type="continuous">
+    <origin
+      xyz="-0.08 -0.08 0.04"
+      rpy="0 0 0" />
+    <parent
+      link="base_link" />
+    <child
+      link="link_wheel_BR" />
+    <axis
+      xyz="0 1 0" />
+  </joint>
+  <link
+    name="camera">
+    <inertial>
+      <origin
+        xyz="-0.0050423 0 0.01"
+        rpy="0 0 0" />
+      <mass
+        value="0.003959" />
+      <inertia
+        ixx="2.6388E-07"
+        ixy="1.0006E-21"
+        ixz="6.9411E-22"
+        iyy="1.6457E-07"
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
Commit message: update md

File: workspace/src/hsa_bot/urdf/hsa_bot.xacro (robot description, xacro)
@@ -327,5 +327,5 @@
   </joint>
   <!--laser_link-->
-  <link name="hokuyo">
+  <link name="laser">
     <collision>
       <origin xyz="0 0 0" rpy="0 0 0"/>
@@ -349,9 +349,9 @@
     </inertial>
   </link>
-  <joint name="hokuyo_joint" type="fixed">
+  <joint name="laser_joint" type="fixed">
     <axis xyz="0 0 0" />
-    <origin xyz="0 0 0.1" rpy="0 0 0"/>
+    <origin xyz="0 0 0.1" rpy="0 0 1.57"/>
     <parent link="base_link"/>
-    <child link="hokuyo"/>
+    <child link="laser"/>
   </joint>
 </robot>

Commit message: update changes

File: workspace/src/hsa_bot/urdf/hsa_bot.xacro (robot description, xacro)
@@ -351,5 +351,5 @@
   <joint name="laser_joint" type="fixed">
     <axis xyz="0 0 0" />
-    <origin xyz="0 0 0.1" rpy="0 0 1.57"/>
+    <origin xyz="0.05 0 0.08" rpy="0 0 -1.57"/>
     <parent link="base_link"/>
     <child link="laser"/>
